File: hardware/sa818-u-carrier/sa818-u-carrier.kicad_pcb (KiCad board)
At the start: 2 copper layers, 0 parts

Commit message: vhf board layout
Other:
- copper layers 2 -> 0
Changed lines of the file:
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@@
-(kicad_pcb
-	(version 20250114)
-	(generator "pcbnew")
-	(generator_version "9.0")
-	(general
-		(thickness 1.6)
-		(legacy_teardrops no)
-	)
-	(paper "A4")
-	(layers
-		(0 "F.Cu" signal)
-		(31 "B.Cu" signal)
-		(32 "B.Adhes" user "B.Adhesive")
-		(33 "F.Adhes" user "F.Adhesive")
-		(34 "B.Paste" user)
-		(35 "F.Paste" user)
-		(36 "B.SilkS" user "B.Silkscreen")
-		(37 "F.SilkS" user "F.Silkscreen")
-		(38 "B.Mask" user "B.Mask")
-		(39 "F.Mask" user "F.Mask")
-		(40 "Dwgs.User" user "User.Drawings")
-		(41 "Cmts.User" user "User.Comments")
-		(42 "Eco1.User" user "User.Eco1")
-		(43 "Eco2.User" user "User.Eco2")
-		(44 "Edge.Cuts" user)
-		(45 "Margin" user)
-		(46 "B.CrtYd" user "B.Courtyard")
-		(47 "F.CrtYd" user "F.Courtyard")
-		(48 "B.Fab" user)
-		(49 "F.Fab" user)
-	)
-	(setup
-		(pad_to_mask_clearance 0)
-		(allow_soldermask_bridges_in_footprints no)
-		(pcbplotparams
-			(layerselection 0x00010fc_ffffffff)
-			(plot_on_all_layers_selection 0x0000000_00000000)
-			(disableapertmacros no)
-			(usegerberextensions no)
-			(usegerberattributes yes)
-			(usegerberadvancedattributes yes)
-			(creategerberjobfile yes)
-			(dashed_line_dash_ratio 12.000000)
-			(dashed_line_gap_ratio 3.000000)
-			(svgprecision 4)
-			(plotframeref no)
-			(viasonmask no)
-			(mode 1)
-			(useauxorigin no)
-			(hpglpennumber 1)
-			(hpglpenspeed 20)
-			(hpglpendiameter 15.000000)
-			(pdf_front_fp_property_popups yes)
-			(pdf_back_fp_property_popups yes)
-			(pdf_metadata yes)
-			(excludeedgelayer yes)
-			(linewidth 0.100000)
-			(plotinvisibletext no)
-			(sketchpadsonfab no)
-			(subtractmaskfromsilk no)
-			(outputformat 1)
-			(mirror no)
-			(drillshape 1)
-			(scaleselection 1)
-			(outputdirectory "")
-		)
-	)
-	(net 0 "")
+(kicad_pcb (version 20241229) (generator "pcbnew") (generator_version "9.0")
 )

Commit message: VHF Carrier Board
Parts:
- added C56: 100nF, Capacitor_SMD:C_0402_1005Metric, F.Cu at (116.5, 76.9)
- added C57: 10uF, Capacitor_SMD:C_0603_1608Metric, F.Cu at (105.6, 76.9)
- added J18: Conn_Coaxial, Connector_Coaxial:SMA_Amphenol_132289_EdgeMount, F.Cu at (126.7, 52.6)
- added J19: Power/Audio, Connector_PinHeader_2.54mm:PinHeader_1x08_P2.54mm_Vertical, F.Cu at (112.0, 87.0)
- added J20: Control/Data, Connector_PinHeader_2.54mm:PinHeader_1x08_P2.54mm_Vertical, F.Cu at (168.0, 87.0)
- added J21: Conn_01x03_Pin, Connector_PinHeader_2.54mm:PinHeader_1x03_P2.54mm_Vertical, F.Cu at (87.0, 53.0)
- added J22: Conn_01x03_Pin, Connector_PinHeader_2.54mm:PinHeader_1x03_P2.54mm_Vertical, F.Cu at (193.0, 53.0)
- added R18: 0, Resistor_SMD:R_0402_1005Metric, F.Cu at (143.0, 87.0)
- added U10: SA818U, VHF_UHF_Modules:VHF_UHF_Module_generic, F.Cu at (140.0, 70.0)
Routing:
- net Net-(J20-Pin_5): track 0.00 -> 65.5 mm
- net Net-(J20-Pin_6): track 0.00 -> 53.0 mm
- net Net-(J19-Pin_3): track 0.00 -> 47.8 mm
- net Net-(J20-Pin_2): track 0.00 -> 42.1 mm, vias 0 -> 2
- net Net-(J20-Pin_3): track 0.00 -> 41.6 mm
- net Net-(J20-Pin_1): track 0.00 -> 38.4 mm, vias 0 -> 2
- net Net-(J19-Pin_5): track 0.00 -> 30.7 mm, vias 0 -> 2
- net Net-(J19-Pin_1): track 0.00 -> 29.4 mm
- net Net-(J20-Pin_4): track 0.00 -> 16.0 mm
- net Net-(J20-Pin_7): track 0.00 -> 10.2 mm
- net Net-(J18-In): track 0.00 -> 8.60 mm
- net GND: vias 0 -> 8
- added copper zone on B.Cu, net GND
- added copper zone on F.Cu, net GND
Other:
- board outline added: 120 x 40 mm
- copper layers 0 -> 2
- board text added: "HAM RADIO VILLAGE SSTV BADGE (VHF) SEND ME YOUR MEMES OR POSE FOR A SELFIE JOIN US! https://hamvillage.org"
- board text added: "HRV SSTV BADGE UHF CARRIER BOARD REV 0.1"
