File: hardware/main_badge/defcon-sstv-badge-clean.kicad_pcb (KiCad board)
At the start: 4 copper layers, 185.7 x 199 mm, 136 parts, among them J1 Conn_01x02, J10 Micro_SD_Card, J11 Mechanical/Grounds, J12 Mechanical/Grounds, J2 USB4105-GF-A, J3 ILI9341 Display Module, J4 Conn_02x09_Odd_Even, J5 SAO1, J6 SAO2, J7 Conn_01x08_Socket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

Commit message: wip routing
Parts:
- moved C10 92.8 mm to (92.0, 169.3)
- moved C13 92.8 mm to (109.6, 163.4)
- moved C14 92.8 mm to (108.3, 152.6)
- moved C21 92.8 mm to (105.7, 82.1)
- moved C22 92.8 mm to (104.8, 85.6)
- moved C26 92.8 mm to (107.3, 106.5)
- moved C27 92.8 mm to (107.3, 113.5)
- moved C30 92.8 mm to (62.9, 35.3)
- moved C36 92.8 mm to (178.6, 44.9)
- moved C39 92.8 mm to (135.4, 129.1)
- moved C4 92.8 mm to (117.1, 98.4)
- moved C40 92.8 mm to (122.5, 129.1)
- moved C41 92.8 mm to (109.7, 129.1)
- moved C42 92.8 mm to (96.9, 129.1)
- moved C43 92.8 mm to (151.2, 142.9)
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Routing:
- net I2C_SDA: track 23.9 -> 280.0 mm, vias 0 -> 2
- net I2C_SCL: track 29.5 -> 259.2 mm, vias 0 -> 2
- net +3V3: track 248.9 -> 74.3 mm, vias 32 -> 10
- net CAM_D5: track 2.06 -> 137.3 mm, vias 0 -> 3
- net CAM_D4: track 0.00 -> 128.0 mm, vias 0 -> 3
- net Net-(U1-~{QSPI_SS}): track 25.8 -> 151.4 mm, vias 0 -> 3
- net CAM_D2: track 124.7 -> 0.00 mm, vias 5 -> 0
- net CAM_D3: track 122.9 -> 0.00 mm, vias 5 -> 0
- net SPI_MOSI: track 76.6 -> 199.1 mm
- net CAM_D6: track 1.95 -> 122.4 mm, vias 0 -> 3
- net CAM_D0: track 118.6 -> 0.00 mm, vias 9 -> 0
- net USB_DM: track 97.0 -> 0.00 mm, vias 3 -> 1
- net SA818_PD: track 18.0 -> 112.2 mm, vias 2 -> 3
- net GND: track 467.3 -> 558.5 mm, vias 59 -> 31
- net DPAD_RIGHT: track 96.3 -> 6.50 mm, vias 1 -> 0
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