File: hardware/main_badge/camera-display.kicad_sch (KiCad schematic)
At the start: 6 parts, among them J3 ILI9341 Display Module, J4 OV2640 Camera Module, Q1 2N7002

Commit message: main board done except for placing LEDs and drawing ears... I think
Parts:
- removed J4: OV2640 Camera Module, Connector_PinSocket_2.54mm:PinSocket_1x18_P2.54mm_Vertical, symbol Connector:Conn_01x18_Socket
- added J4: Conn_02x09_Odd_Even, Connector_PinSocket_2.54mm:PinSocket_2x09_P2.54mm_Vertical, symbol Connector_Generic:Conn_02x09_Odd_Even
Connections:
- net +3V3: now also J4.2 (Pin_2)
- net CAM_D0: now also J4.7 (Pin_7)
- net CAM_D1: now also J4.10 (Pin_10)
- net CAM_D2: now also J4.9 (Pin_9)
- net CAM_D3: now also J4.12 (Pin_12)
- net CAM_D4: now also J4.11 (Pin_11)
- net CAM_D5: now also J4.14 (Pin_14)
- net CAM_D6: now also J4.13 (Pin_13)
- net CAM_D7: now also J4.16 (Pin_16)
- net CAM_HREF: now also J4.6 (Pin_6)
- net CAM_PCLK: now also J4.15 (Pin_15)
- net CAM_VSYNC: now also J4.4 (Pin_4)
- net GND: now also J4.1 (Pin_1)
- net I2C_SCL: now also J4.3 (Pin_3)
- net I2C_SDA: now also J4.5 (Pin_5)
- net at R12.1: now also J4.8 (Pin_8)
- net at R13.1: now also J4.17 (Pin_17)
- no-connect marks 5 -> 6
Other:
- moved on the sheet: R13

Commit message: more routing, 29 to go...
Connections:
- net GND: now also Q1.2 (S); no longer Q1.3 (D)
- net at J3.8 (Pin_8): now also Q1.3 (D); no longer Q1.2 (S)
Other:
- moved on the sheet: Q1
Changed lines of the file:
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@@
 	(symbol
 		(lib_id "Transistor_FET:2N7002")
-		(at 187.96 45.72 90)
+		(at 187.96 45.72 270)
+		(mirror x)
 		(unit 1)
 		(exclude_from_sim no)
@@
 		(on_board yes)
 		(dnp no)
-		(fields_autoplaced yes)
 		(property "Reference" "Q1"
 			(at 187.96 36.83 90)
@@
 		)
 		(property "Footprint" "Package_TO_SOT_SMD:SOT-23"
-			(at 189.865 40.64 0)
+			(at 186.055 40.64 0)
 			(effects
 				(font
@@
 		)
 		(property "Datasheet" "https://www.onsemi.com/pub/Collateral/NDS7002A-D.PDF"
-			(at 191.77 40.64 0)
+			(at 184.15 40.64 0)
 			(effects
 				(font
