File: hardware/main_badge/defcon-sstv-badge.kicad_pcb (KiCad board)
At the start: 4 copper layers, 185.7 x 199 mm, 136 parts, among them J1 Conn_01x02, J10 Micro_SD_Card, J11 Mechanical/Grounds, J12 Mechanical/Grounds, J2 USB4105-GF-A, J3 ILI9341 Display Module, J4 Conn_02x09_Odd_Even, J5 SAO1, J6 SAO2, J7 Conn_01x08_Socket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

Commit message: more routing, 29 to go...
Parts:
- moved C19 30.8 mm to (40.1, 23.0), turned to 180 degrees
- moved C_OUT1 9.69 mm to (31.3, 85.7), turned to 90 degrees
- moved R15 2.94 mm to (68.4, 47.2), turned to 90 degrees
- moved R16 2.91 mm to (71.3, 47.2), turned to 90 degrees
- moved R14 1.98 mm to (65.3, 47.2), turned to 90 degrees
- moved C22 0.95 mm to (40.1, 20.1)
- moved C16 0.35 mm to (36.4, 95.4)
Connections:
- Q1 pad 2: Net-(J3-Pin_8) -> GND
- Q1 pad 3: GND -> Net-(J3-Pin_8)
Routing:
- net I2C_SDA: track 23.9 -> 289.0 mm, vias 0 -> 6
- net I2C_SCL: track 29.5 -> 280.5 mm, vias 0 -> 8
- net USB_DP: track 0.00 -> 221.8 mm, vias 0 -> 3
- net CAM_D5: track 2.06 -> 174.1 mm, vias 0 -> 9
- net Net-(U1-~{QSPI_SS}): track 25.8 -> 160.6 mm, vias 0 -> 3
- net CAM_D4: track 0.00 -> 112.4 mm, vias 0 -> 4
- net CAM_VSYNC: track 0.44 -> 106.6 mm, vias 0 -> 6
- net SA818_PD: track 18.0 -> 123.4 mm, vias 2 -> 8
- net SPI_MISO: track 103.5 -> 189.7 mm, vias 2 -> 4
- net SD_CS: track 0.00 -> 81.9 mm, vias 0 -> 3
- net SAO2_GPIO1: track 0.00 -> 76.8 mm, vias 0 -> 4
- net SPI_SCK: track 88.5 -> 161.8 mm, vias 1 -> 3
- net DISP_BL: track 0.00 -> 71.5 mm, vias 0 -> 4
- net SPI_MOSI: track 76.6 -> 147.3 mm, vias 2 -> 3
- net SAO2_GPIO2: track 0.00 -> 63.0 mm, vias 0 -> 4
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
Commit message: routing. 2 nodes to go...
Parts:
- turned C16 to -90 degrees
Routing:
- net SAO1_GPIO2: track 0.00 -> 140.3 mm, vias 0 -> 5
- net CAM_D6: track 1.95 -> 140.4 mm, vias 0 -> 11
- net CAM_D7: track 1.97 -> 128.2 mm, vias 0 -> 9
- net CAM_PCLK: track 3.09 -> 118.7 mm, vias 0 -> 9
- net GND: track 494.0 -> 577.9 mm, vias 69 -> 74
- net USB_DM: track 95.9 -> 142.7 mm, vias 3 -> 5
- net VBUS: track 40.0 -> 75.6 mm, vias 4 -> 9
- net CAM_VSYNC: track 106.6 -> 141.6 mm, vias 6 -> 8
- net Net-(J2-DP1): track 2.31 -> 33.3 mm, vias 0 -> 2
- net SD_CS: track 81.9 -> 64.1 mm
- net +3V3: track 304.1 -> 321.2 mm, vias 39 -> 43
- net Net-(J2-DN1): track 20.7 -> 29.2 mm, vias 2 -> 3
- net USB_DP: track 221.8 -> 213.7 mm
- net CAM_D4: track 112.4 -> 119.8 mm, vias 4 -> 6
- net DPAD_DOWN: track 72.5 -> 79.3 mm
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
Commit message: all traces complete, but lots of DRC warnings to fix
Routing:
- net SAO1_GPIO1: track 0.00 -> 69.9 mm, vias 0 -> 6
- net +3V3: track 321.2 -> 322.6 mm, vias 43 -> 44
- net Net-(U1-XIN): track 6.35 -> 7.26 mm
- net (no net): track 0.00 -> 0.10 mm, vias 0 -> 1

Commit message: connect J7 pin 8 to GND
Connections:
- J7 pad 8: unconnected-(J7-Pin_8-Pad8) -> GND
Routing:
- net GND: track 577.9 -> 580.1 mm, vias 74 -> 75

Commit message: main board finished, no DRC errors
Connections:
- U5 pad 12: (no net) -> GND
- U5 pad 13: (no net) -> GND
- U5 pad 14: (no net) -> GND
- U5 pad 15: (no net) -> GND
Routing:
- net I2C_SCL: track 281.1 -> 276.7 mm
- net DISP_RST: track 73.3 -> 71.0 mm
- net SPI_MISO: track 189.7 -> 190.7 mm
- net AIRPLANE: track 148.5 -> 147.9 mm
- net SPI_MOSI: track 147.2 -> 147.8 mm
- net CAM_D6: track 140.4 -> 141.0 mm
- net CAM_D5: vias 8 -> 7
- net VSYS: vias 5 -> 4
